Commit message: Update simpleobstacle.urdf

File: simple_driving/resources/simpleobstacle.urdf (robot description, URDF)
Before this commit: robot simpleobstacle, 1 links, 0 joints
Links:
- link base_link: geometry visual cylinder length=1 radius=0.1

Commit message: Update simpleobstacle.urdf

File: simple_driving/resources/simpleobstacle.urdf (robot description, URDF)
Before this commit: robot simpleobstacle, 1 links, 0 joints
Links:
- link base_link: geometry visual cylinder length=1 radius=0.3
